Commit message: change robot model to a 4-wheeled differencial derive

File: src/sdnt_robot_description/src/description/sdnt_robot_description.urdf (robot description, URDF)
Before this commit: robot sdnt_robot, 7 links, 6 joints
Links:
- removed link front_caster
- removed link imu_link
Joints:
- removed joint base_joint
- removed joint caster_joint
- removed joint imu_joint
- added joint base_footprint_joint: type fixed, parent base_link, child base_footprint, origin xyz=0 0 ${-(wheel_radius + 0.02)}
- joint camera_joint: origin xyz=0.215 0 0.05 rpy=0 0 0 -> xyz=${camera_x_forward} 0 ${camera_height}
- joint lidar_joint: origin xyz=0 0 0.14 rpy=0 0 0 -> xyz=0 0 ${lidar_height}
